Commit message: Update robot.urdf - added camera link and wheels onto robot simulation

File: src/robot_bringup/urdf/robot.urdf (robot description, URDF)
Before this commit: robot simple_robot, 2 links, 1 joints
Links:
- added link left_wheel; visual cylinder length=0.05 radius=0.06
- added link right_wheel; visual cylinder length=0.05 radius=0.06
- added link world
- link base_link: geometry visual box size=0.40 0.25 0.05
- link camera_link: geometry visual box size=0.06 0.04 0.03
Joints:
- removed joint base_to_camera
- added joint camera_joint: type fixed, parent base_link, child camera_link, origin xyz=0.2 0 0.1 rpy=0 0 0
- added joint left_wheel_joint: type fixed, parent base_link, child left_wheel, origin xyz=0 0.12 0.06 rpy=0 0 0
- added joint right_wheel_joint: type fixed, parent base_link, child right_wheel, origin xyz=0 -0.12 0.06 rpy=0 0 0
- added joint world: type fixed, parent world, child base_link, origin xyz=0 0 0.5 rpy=0 0 0

Commit message: Update robot.urdf

File: src/robot_bringup/urdf/robot.urdf (robot description, URDF)
Before this commit: robot simple_robot, 5 links, 4 joints
Links:
- added link camera_link_optical
Joints:
- added joint camera_optical_joint: type fixed, parent camera_link, child camera_link_optical, origin xyz=0 0 0 rpy=-1.5708 0 -1.5708
